Commit message: - adding more plotJuggler plots

File: src/my_robot_description/urdf/cubic_doggo_legB.xacro (robot description, xacro)
@@ -222,5 +222,5 @@
         <visual>
             <geometry>
-                <mesh filename="package://my_robot_description/mesh/CADv2/calfFeet.stl" scale="0.001 0.001 0.001"/>
+                <mesh filename="package://my_robot_description/mesh/CADv2/calfFeetSpring.stl" scale="0.001 0.001 0.001"/>
             </geometry>
             <material name="purple"/>

File: src/my_robot_description/urdf/cubic_doggo_legF.xacro (robot description, xacro)
@@ -222,5 +222,5 @@
         <visual>
             <geometry>
-                <mesh filename="package://my_robot_description/mesh/CADv2/calfFeet.stl" scale="0.001 0.001 0.001"/>
+                <mesh filename="package://my_robot_description/mesh/CADv2/calfFeetSpring.stl" scale="0.001 0.001 0.001"/>
             </geometry>
             <material name="purple"/>
